File: WeMos-shield.brd (EAGLE design)
At the start: 33 x 25.4 mm, 23 parts, among them Q1 N-MOS

Commit message: Version 1.1
Parts:
- added U$1, U$2: PAD, _c2h:PAD-JUMPER-SWAP
Connections:
- new net V+J: I2C_OLED.1, U$2.3
- new net V+O: I2C_OLED1.1, U$1.3
- new net V-J: I2C_OLED.2, U$2.2
- new net V-O: I2C_OLED1.2, U$1.2
- net 3V3: now also U$1.4, U$1.44, U$2.4, U$2.44; no longer I2C_OLED.1, I2C_OLED1.1
- net GND: now also U$1.1, U$1.11, U$2.1, U$2.11; no longer I2C_OLED.2, I2C_OLED1.2
Routing:
- net V-O: track 0.00 -> 7.38 mm
- net V+O: track 0.00 -> 5.75 mm
- net V-J: track 0.00 -> 4.75 mm
- net V+J: track 0.00 -> 4.75 mm
- net GND: track 2.54 -> 5.21 mm, vias 0 -> 1
- net SDA: track 55.4 -> 56.8 mm, vias 0 -> 1
- net SCL: track 49.4 -> 50.5 mm, vias 0 -> 1
- net 3V3: track 81.6 -> 81.9 mm, vias 2 -> 1
Other:
- board size 33 x 25.4 mm -> 33.2 x 25.7 mm
- board text added: "V1.1"
- board text removed: "I2C Pullups"
